Commit message: Fully Fixed URDF, will maybe replace bulky models with primitives

File: install/soarm_description/share/soarm_description/urdf/soarm.urdf.xacro (robot description, xacro)
@@ -177,5 +177,5 @@
     <visual>
       <!--       <origin xyz="-0.065085 0.012 0.0182" rpy="3.14159 -0 -1.30911e-30"/> -->
-      <origin xyz="0 0 0" rpy="3.14159 0 ${3*PI/2}"/>
+      <origin xyz="0.01 .065 0" rpy="3.14159 0 ${3*PI/2}"/>
       <geometry>
         <mesh filename="package://soarm_description/meshes/Upper_arm_SO101.stl" scale="0.001 0.001 0.001"/>
@@ -186,5 +186,5 @@
     </visual>
     <collision>
-      <origin xyz="0 0 0" rpy="3.14159 0 ${3*PI/2}"/>
+      <origin xyz="0.01 .065 0" rpy="3.14159 0 ${3*PI/2}"/>
       <geometry>
         <mesh filename="package://soarm_description/meshes/Upper_arm_SO101.stl" scale="0.001 0.001 0.001"/>
@@ -201,5 +201,6 @@
     <!-- Part Under_arm_SO101 -->
     <visual>
-      <origin xyz="-0.0648499 -0.032 0.0182" rpy="3.14159 -0 6.67202e-31"/>
+        <!-- <origin xyz="-0.0648499 -0.032 0.0182" rpy="3.14159 -0 6.67202e-31"/> -->
+      <origin xyz="-0.0648499 -0.032 0" rpy="3.14159 -0 0"/>
       <geometry>
         <mesh filename="package://soarm_description/meshes/Under_arm_SO101.stl" scale="0.001 0.001 0.001"/>
@@ -210,5 +211,6 @@
     </visual>
     <collision>
-      <origin xyz="-0.0648499 -0.032 0.0182" rpy="3.14159 -0 6.67202e-31"/>
+    <!--       <origin xyz="-0.0648499 -0.032 0.0182" rpy="3.14159 -0 6.67202e-31"/> -->
+      <origin xyz="-0.0648499 -0.032 0" rpy="3.14159 -0 0"/>
       <geometry>
         <mesh filename="package://soarm_description/meshes/Under_arm_SO101.stl" scale="0.001 0.001 0.001"/>
@@ -216,5 +218,5 @@
     </collision>
     <!-- Part Motor_holder_SO101_Wrist -->
-    <visual>
+    <!-- <visual>
       <origin xyz="-0.0648499 -0.032 0.018" rpy="-3.14159 -2.55351e-15 -2.56146e-31"/>
       <geometry>
@@ -230,5 +232,5 @@
         <mesh filename="package://soarm_description/meshes/Motor_holder_SO101_Wrist.stl" scale="0.001 0.001 0.001"/>
       </geometry>
-    </collision>
+    </collision> -->
     <!-- Part sts3215_03a_v1_4 -->
     <!-- <visual>
@@ -273,5 +275,6 @@
     <!-- Part Wrist_Roll_Pitch_SO101 -->
     <visual>
-      <origin xyz="0 -0.028 0.0181" rpy="-1.5708 -1.5708 0"/>
+      <!--<origin xyz="0 -0.028 0.0181" rpy="-1.5708 -1.5708 0"/> -->
+      <origin xyz="0 -0.028 0" rpy="-1.5708 -1.5708 0"/>
       <geometry>
         <mesh filename="package://soarm_description/meshes/Wrist_Roll_Pitch_SO101.stl" scale="0.001 0.001 0.001"/>
@@ -282,5 +285,6 @@
     </visual>
     <collision>
-      <origin xyz="0 -0.028 0.0181" rpy="-1.5708 -1.5708 0"/>
+      <!--<origin xyz="0 -0.028 0.0181" rpy="-1.5708 -1.5708 0"/> -->
+      <origin xyz="0 -0.028 0" rpy="-1.5708 -1.5708 0"/>
       <geometry>
         <mesh filename="package://soarm_description/meshes/Wrist_Roll_Pitch_SO101.stl" scale="0.001 0.001 0.001"/>
@@ -313,5 +317,5 @@
     <!-- Part Wrist_Roll_Follower_SO101 -->
     <visual>
-      <origin xyz="0 -0.000218214 0.000949706" rpy="-3.14159 -5.55112e-17 0"/>
+      <origin xyz="0 0 0" rpy="-3.14159 0 0"/>
       <geometry>
         <mesh filename="package://soarm_description/meshes/Wrist_Roll_Follower_SO101.stl" scale="0.001 0.001 0.001"/>
@@ -322,5 +326,5 @@
     </visual>
     <collision>
-      <origin xyz="0 -0.000218214 0.000949706" rpy="-3.14159 -5.55112e-17 0"/>
+      <origin xyz="0 0 0" rpy="-3.14159 0 0"/>
       <geometry>
         <mesh filename="package://soarm_description/meshes/Wrist_Roll_Follower_SO101.stl" scale="0.001 0.001 0.001"/>
@@ -352,5 +356,5 @@
     <!-- Part Moving_Jaw_SO101 -->
     <visual>
-      <origin xyz="-5.55112e-17 0 0.0189" rpy="9.53145e-17 6.93889e-18 1.24077e-24"/>
+      <origin xyz="0 0 0" rpy="0 0 0"/>
       <geometry>
         <mesh filename="package://soarm_description/meshes/Moving_Jaw_SO101.stl" scale="0.001 0.001 0.001"/>
@@ -361,5 +365,5 @@
     </visual>
     <collision>
-      <origin xyz="-5.55112e-17 0 0.0189" rpy="9.53145e-17 6.93889e-18 1.24077e-24"/>
+      <origin xyz="0 0 0" rpy="0 0 0"/>
       <geometry>
         <mesh filename="package://soarm_description/meshes/Moving_Jaw_SO101.stl" scale="0.001 0.001 0.001"/>
@@ -369,5 +373,5 @@
   <!-- Joint from gripper to Moving_Jaw_SO101 -->
   <joint name="gripper" type="revolute">
-    <origin xyz="0.0202 0.0188 -0.0234" rpy="1.5708 -5.24284e-08 -1.41553e-15"/>
+    <origin xyz="0.0202 0 -0.0234" rpy="1.5708 -5.24284e-08 -1.41553e-15"/>
     <parent link="gripper"/>
     <child link="Moving_Jaw_SO101"/>
@@ -377,5 +381,5 @@
   <!-- Joint from wrist to gripper -->
   <joint name="wrist_roll" type="revolute">
-    <origin xyz="2.77556e-16 -0.0611 0.0181" rpy="1.5708 0.0486795 3.14159"/>
+    <origin xyz="0 -0.0611 0.0181" rpy="1.5708 0.0486795 3.14159"/>
     <parent link="wrist"/>
     <child link="gripper"/>
@@ -385,5 +389,5 @@
   <!-- Joint from lower_arm to wrist -->
   <joint name="wrist_flex" type="revolute">
-    <origin xyz="-0.1349 0.0052 8.44651e-17" rpy="4.02456e-15 8.67362e-16 -1.5708"/>
+    <origin xyz="-0.1349 0.004 0" rpy="4.02456e-15 8.67362e-16 -1.5708"/>
     <parent link="lower_arm"/>
     <child link="wrist"/>
@@ -393,5 +397,5 @@
   <!-- Joint from upper_arm to lower_arm -->
   <joint name="elbow_flex" type="revolute">
-    <origin xyz="-0.11257 -0.028 2.09886e-16" rpy="-3.63608e-16 8.74301e-16 1.5708"/>
+    <origin xyz="-0.029 .113 0.004" rpy="0 0 ${PI/2}"/>
     <parent link="upper_arm"/>
     <child link="lower_arm"/>
