Commit message: Working Sweep

File: src/soarm_description/urdf/soarm.urdf.xacro (robot description, xacro)
@@ -275,7 +275,12 @@
     <child link="Moving_Jaw_SO101"/>
     <axis xyz="0 0 1"/>
-    <limit effort="10" velocity="10" lower="-0.174533" upper="1.74533"/>
-    <!-- <limit effort="10" velocity="10" lower="${1300*RAD_CONV}" upper="${2800*RAD_CONV}"/> -->
-  </joint>
+    <!-- is_sim true is Gazebo, false is live -->
+    <xacro:if value="$(arg is_sim)">
+      <limit effort="10" velocity="10" lower="-0.174533" upper="1.74533"/>
+    </xacro:if>
+    <xacro:unless value="$(arg is_sim)">
+      <limit effort="10" velocity="10" lower="${1300*RAD_CONV}" upper="${2800*RAD_CONV}"/>
+    </xacro:unless>
+    </joint>
   <!-- Joint from wrist to gripper -->
   <joint name="wrist_roll" type="revolute">
@@ -284,7 +289,11 @@
     <child link="gripper"/>
     <axis xyz="0 0 1"/>
-    <limit effort="10" velocity="10" lower="${-7*PI/8}" upper="${7*PI/8}"/>
-    <!-- <limit effort="10" velocity="10" lower="${430*RAD_CONV}" upper="${4070*RAD_CONV}"/> -->
-  </joint>
+    <xacro:if value="$(arg is_sim)">
+      <limit effort="10" velocity="10" lower="${-7*PI/8}" upper="${7*PI/8}"/>
+    </xacro:if>
+    <xacro:unless value="$(arg is_sim)">
+      <limit effort="10" velocity="10" lower="${430*RAD_CONV}" upper="${4070*RAD_CONV}"/>
+    </xacro:unless>
+    </joint>
   <!-- Joint from lower_arm to wrist -->
   <joint name="wrist_flex" type="revolute">
@@ -293,7 +302,10 @@
     <child link="wrist"/>
     <axis xyz="0 0 1"/>
-    <limit effort="10" velocity="10" lower="-1.2" upper="1.2"/>
-    <!-- <limit effort="10" velocity="10" lower="${-PI/2}" upper="${PI/2}"/> -->
-    <!-- <limit effort="10" velocity="10" lower="${430*RAD_CONV}" upper="${2750*RAD_CONV}"/> -->
+    <xacro:if value="$(arg is_sim)">
+      <limit effort="10" velocity="10" lower="-1.2" upper="1.2"/>
+    </xacro:if>
+    <xacro:unless value="$(arg is_sim)">
+      <limit effort="10" velocity="10" lower="${1200*RAD_CONV}" upper="${3200*RAD_CONV}"/>
+    </xacro:unless>
   </joint>
   <!-- Joint from upper_arm to lower_arm -->
@@ -303,28 +315,36 @@
     <child link="lower_arm"/>
     <axis xyz="0 0 1"/>
-    <limit effort="10" velocity="10" lower="${-PI}" upper="0"/>
-    <!-- <limit effort="10" velocity="10" lower="${-5*PI/9}" upper="${PI/2}"/> -->
-    <!-- <limit effort="10" velocity="10" lower="${500*RAD_CONV}" upper="${2600*RAD_CONV}"/> -->
-  </joint>
+    <xacro:if value="$(arg is_sim)">
+      <limit effort="10" velocity="10" lower="${-PI}" upper="0"/>
+    </xacro:if>
+    <xacro:unless value="$(arg is_sim)">
+      <limit effort="10" velocity="10" lower="${500*RAD_CONV}" upper="${2600*RAD_CONV}"/>
+    </xacro:unless>
+    </joint>
   <!-- Joint from shoulder to upper_arm -->
   <joint name="shoulder_lift" type="revolute">
-<!-- <origin xyz="-0.0303992 -0.0182778 -0.0542" rpy="-1.5708 -1.5708 0"/> -->
     <origin xyz="-0.03138 0 -0.072" rpy="${-PI/2} ${-PI/2} 0"/>
     <parent link="shoulder"/>
     <child link="upper_arm"/>
     <axis xyz="0 0 1"/>
-    <limit effort="10" velocity="10" lower="-0.3" upper="${PI}"/>
-    <!-- <limit effort="10" velocity="10" lower="${-5*PI/9}" upper="${5*PI/9}"/> -->
-    <!-- <limit effort="10" velocity="10" lower="${850*RAD_CONV}" upper="${3500*RAD_CONV}"/> -->
-  </joint>
+    <xacro:if value="$(arg is_sim)">
+      <limit effort="10" velocity="10" lower="-0.3" upper="${PI}"/>
+    </xacro:if>
+    <xacro:unless value="$(arg is_sim)">
+      <limit effort="10" velocity="10" lower="${850*RAD_CONV}" upper="${3500*RAD_CONV}"/>
+    </xacro:unless>
+    </joint>
   <!-- Joint from base to shoulder -->
   <joint name="shoulder_pan" type="revolute">
-    <!-- Y+.45 Z <origin xyz="-0.124202 -0.168068 0.0948817" rpy="3.14159 4.18253e-17 -3.14159"/> -->
     <origin xyz="0.04572 0 0.048" rpy="${PI} 0 ${-PI}"/>
     <parent link="base"/>
     <child link="shoulder"/>
     <axis xyz="0 0 1"/>
-    <limit effort="10" velocity="10" lower="${-3*PI/5}" upper="${3*PI/5}"/>
-    <!-- <limit effort="10" velocity="10" lower="${1130*RAD_CONV)" upper="(3730*RAD_CONV)"/> -->
-  </joint>
+    <xacro:if value="$(arg is_sim)">
+      <limit effort="10" velocity="10" lower="${-3*PI/5}" upper="${3*PI/5}"/>
+    </xacro:if>
+    <xacro:unless value="$(arg is_sim)">
+      <limit effort="10" velocity="10" lower="${1130*RAD_CONV}" upper="${3730*RAD_CONV}"/>
+    </xacro:unless>
+    </joint>
 </robot>

File: src/soarm_description/urdf/soarm_ros2_control.xacro (robot description, xacro)
@@ -2,14 +2,9 @@
 <robot xmlns:xacro="http://www.ros.org/wiki/xacro"  name="soarm">
     <!-- Wrap everything in a macro -->
+    <xacro:arg name="is_sim" default="true" />
     <xacro:macro name="soarm_ros2_control" params="is_sim">
-        <xacro:arg name="is_sim" default="true" />
-        <!-- Convert arg into property -->
         <xacro:property name="is_sim_prop" value="$(arg is_sim)"/>
         <xacro:property name="PI" value="3.14159"/>
         <xacro:property name="RAD_CONV" value="0.001533979"/>
-        <!-- Test with bypassing Gazebo Plugins -->
-        <!-- <hardware>
-            <plugin>mock_components/GenericSystem</plugin>
-        </hardware> -->
         <ros2_control name="SO_ARM101" type="system">
             <!-- ros2_control Gazebo -->
@@ -23,12 +18,25 @@
                 <hardware>
                     <plugin>feetech_ros2_driver/FeetechHardwareInterface</plugin>
-                    <param name="port">/dev/ttyACM0</param>
+                    <param name="usb_port">/dev/ttyACM0</param>
+                    <param name="baud_rate">1000000</param>
                 </hardware>
             </xacro:unless>
             <joint name="gripper_joint">
+                <xacro:unless value="${is_sim_prop}">
+                    <param name="initial_position">0</param>
+                    <param name="id">12</param>
+                    <param name="p_cofficient">32</param>
+                    <!-- <param name="offset">0</param> -->
+                </xacro:unless>
                 <!--Send commands to hardware-->
                 <command_interface name="position">
-                    <param name="min">-0.174533</param>
-                    <param name="max">0.174533</param>
+                    <xacro:if value="${is_sim_prop}">
+                        <param name="min">-0.174533</param>
+                        <param name="max">0.174533</param>
+                    </xacro:if>
+                    <xacro:unless value="${is_sim_prop}">
+                        <param name="min">${1300*RAD_CONV}</param>
+                        <param name="max">${2800*RAD_CONV}</param>
+                    </xacro:unless>
                 </command_interface>
                 <!--Read Feedback from hardware-->
@@ -37,7 +45,19 @@
             </joint>
             <joint name="wrist_roll">
+                <xacro:unless value="${is_sim_prop}">
+                    <param name="initial_position">0</param>
+                    <param name="id">11</param>
+                    <param name="p_cofficient">32</param>
+                    <!-- <param name="offset">0</param> -->
+                </xacro:unless>
                 <command_interface name="position">
-                    <param name="min">${-7*PI/8}</param>
-                    <param name="max">${7*PI/8}</param>
+                    <xacro:if value="${is_sim_prop}">
+                        <param name="min">${-7*PI/8}</param>
+                        <param name="max">${7*PI/8}</param>
+                    </xacro:if>
+                    <xacro:unless value="${is_sim_prop}">
+                        <param name="min">${430*RAD_CONV}</param>
+                        <param name="max">${4070*RAD_CONV}</param>
+                    </xacro:unless>
                 </command_interface>
                 <state_interface name="position"/>
@@ -45,9 +65,19 @@
             </joint>
             <joint name="wrist_flex">
+                <xacro:unless value="${is_sim_prop}">
+                    <param name="initial_position">0</param>
+                    <param name="id">10</param>
+                    <param name="p_cofficient">32</param>
+                    <!-- <param name="offset">0</param> -->
+                </xacro:unless>
                 <command_interface name="position">
-                    <!-- <param name="min">${-PI/2}</param>
-                    <param name="max">${PI/2}</param> -->
-                    <param name="min">-1.2</param>
-                    <param name="max">1.2</param>
+                    <xacro:if value="${is_sim_prop}">
+                        <param name="min">-1.2</param>
+                        <param name="max">1.2</param>
+                    </xacro:if>
+                    <xacro:unless value="${is_sim_prop}">
+                        <param name="min">${1200*RAD_CONV}</param>
+                        <param name="max">${3200*RAD_CONV}</param>
+                    </xacro:unless>
                 </command_interface>
                 <state_interface name="position"/>
@@ -55,9 +85,19 @@
             </joint>
             <joint name="elbow_flex">
+                <xacro:unless value="${is_sim_prop}">
+                    <param name="initial_position">0</param>
+                    <param name="id">9</param>
+                    <param name="p_cofficient">32</param>
+                    <!-- <param name="offset">0</param> -->
+                </xacro:unless>
                 <command_interface name="position">
-                    <!-- <param name="min">${-5*PI/9}</param>
-                    <param name="max">${PI/2}</param> -->
-                    <param name="min">${-PI}</param>
-                    <param name="max">0</param>
+                    <xacro:if value="${is_sim_prop}">
+                        <param name="min">${-PI}</param>
+                        <param name="max">0</param>
+                    </xacro:if>
+                    <xacro:unless value="${is_sim_prop}">
+                        <param name="min">${500*RAD_CONV}</param>
+                        <param name="max">${2600*RAD_CONV}</param>
+                    </xacro:unless>
                 </command_interface>
                 <state_interface name="position"/>
@@ -65,9 +105,19 @@
             </joint>
             <joint name="shoulder_lift">
+                <xacro:unless value="${is_sim_prop}">
+                    <param name="initial_position">0</param>
+                    <param name="id">8</param>
+                    <param name="p_cofficient">32</param>
+                    <!-- <param name="offset">0</param> -->
+                </xacro:unless>
                 <command_interface name="position">
-                    <!-- <param name="min">${-5*PI/9}</param>
-                    <param name="max">${5*PI/9}</param> -->
-                    <param name="min">-0.3</param>
-                    <param name="max">${PI}</param>
+                    <xacro:if value="${is_sim_prop}">
+                        <param name="min">-0.3</param>
+                        <param name="max">${PI}</param>
+                    </xacro:if>
+                    <xacro:unless value="${is_sim_prop}">
+                        <param name="min">${850*RAD_CONV}</param>
+                        <param name="max">${3500*RAD_CONV}</param>
+                    </xacro:unless>
                 </command_interface>
                 <state_interface name="position"/>
@@ -75,7 +125,19 @@
             </joint>
             <joint name="shoulder_pan">
+                <xacro:unless value="${is_sim_prop}">
+                    <param name="initial_position">0</param>
+                    <param name="id">7</param>
+                    <param name="p_cofficient">32</param>
+                    <!-- <param name="offset">0</param> -->
+                </xacro:unless>
                 <command_interface name="position">
-                    <param name="min">${-3*PI/5}</param>
-                    <param name="max">${3*PI/5}</param>
+                    <xacro:if value="${is_sim_prop}">
+                        <param name="min">${-3*PI/5}</param>
+                        <param name="max">${3*PI/5}</param>
+                    </xacro:if>
+                    <xacro:unless value="${is_sim_prop}">
+                        <param name="min">${1130*RAD_CONV}</param>
+                        <param name="max">${3730*RAD_CONV}</param>
+                    </xacro:unless>
                 </command_interface>
                 <state_interface name="position"/>
